File: hardware/eagle/Prototype1.brd (EAGLE design)
At the start: 100 x 80 mm, 26 parts, among them U1 ARDUINO_SHIELDLABEL

Commit message: logo ideas
Routing:
- net N$42: track 0.00 -> 24.0 mm
- net N$45: track 0.00 -> 19.1 mm
- net N$40: track 0.00 -> 17.8 mm
- net N$34: track 0.00 -> 17.7 mm
- net N$41: track 0.00 -> 17.4 mm
- net N$33: track 0.00 -> 15.5 mm
- net N$48: track 0.00 -> 14.0 mm
- net N$44: track 0.00 -> 13.5 mm
- net N$32: track 0.00 -> 12.3 mm
- net N$47: track 0.00 -> 12.2 mm
- net N$38: track 0.00 -> 11.2 mm
- net N$35: track 0.00 -> 10.9 mm
- net N$46: track 0.00 -> 9.04 mm
- net N$43: track 0.00 -> 7.25 mm
- added copper zone on layer 1, net N$49
Changed lines of the file:
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@@
 <wire x1="39.37" y1="66.675" x2="35.56" y2="66.675" width="0.6096" layer="1"/>
 <wire x1="35.56" y1="66.675" x2="34.925" y2="66.04" width="0.6096" layer="1"/>
-<wire x1="31.75" y1="64.135" x2="33.655" y2="66.04" width="0.4064" layer="1"/>
+<wire x1="31.75" y1="64.135" x2="33.655" y2="66.04" width="0.4064" layer="1" curve="-90"/>
 <wire x1="34.925" y1="66.04" x2="33.655" y2="66.04" width="0.6096" layer="1"/>
 </signal>
@@
 <wire x1="36.195" y1="65.405" x2="35.56" y2="64.77" width="0.6096" layer="1"/>
 <wire x1="35.56" y1="64.77" x2="34.29" y2="64.77" width="0.6096" layer="1"/>
-<wire x1="34.29" y1="64.77" x2="32.385" y2="62.865" width="0.4064" layer="1"/>
+<wire x1="34.29" y1="64.77" x2="32.385" y2="62.865" width="0.4064" layer="1" curve="90"/>
 <wire x1="32.385" y1="62.865" x2="32.385" y2="55.88" width="0.4064" layer="1"/>
 <wire x1="32.385" y1="55.88" x2="24.765" y2="48.26" width="0.4064" layer="1"/>
@@
 <wire x1="24.765" y1="50.8" x2="31.115" y2="57.15" width="0.4064" layer="1"/>
 <wire x1="31.115" y1="57.15" x2="31.115" y2="65.405" width="0.4064" layer="1"/>
-<wire x1="31.115" y1="65.405" x2="33.02" y2="67.31" width="0.4064" layer="1"/>
+<wire x1="31.115" y1="65.405" x2="33.02" y2="67.31" width="0.4064" layer="1" curve="-90"/>
 <wire x1="33.02" y1="67.31" x2="33.655" y2="67.945" width="0" layer="19" extent="1-16"/>
 <wire x1="47.345" y1="55.88" x2="45.085" y2="55.88" width="0.6096" layer="1"/>
@@
 <wire x1="24.765" y1="52.07" x2="30.48" y2="57.785" width="0.4064" layer="1"/>
 <wire x1="30.48" y1="57.785" x2="30.48" y2="66.675" width="0.4064" layer="1"/>
-<wire x1="30.48" y1="66.675" x2="32.385" y2="68.58" width="0.4064" layer="1"/>
+<wire x1="30.48" y1="66.675" x2="32.385" y2="68.58" width="0.4064" layer="1" curve="-90"/>
 <wire x1="32.385" y1="68.58" x2="33.655" y2="69.85" width="0" layer="19" extent="1-16"/>
 <wire x1="47.845" y1="58.42" x2="45.085" y2="58.42" width="0.6096" layer="1"/>
@@
 <wire x1="33.655" y1="70.485" x2="33.02" y2="69.85" width="0.6096" layer="1"/>
 <wire x1="33.02" y1="69.85" x2="31.75" y2="69.85" width="0.6096" layer="1"/>
-<wire x1="31.75" y1="69.85" x2="29.845" y2="67.945" width="0.4064" layer="1"/>
+<wire x1="31.75" y1="69.85" x2="29.845" y2="67.945" width="0.4064" layer="1" curve="90" cap="flat"/>
 </signal>
 <signal name="N$14">
@@
 <wire x1="33.02" y1="71.755" x2="32.385" y2="71.12" width="0.6096" layer="1"/>
 <wire x1="32.385" y1="71.12" x2="31.115" y2="71.12" width="0.6096" layer="1"/>
-<wire x1="29.21" y1="69.215" x2="31.115" y2="71.12" width="0.4064" layer="1"/>
+<wire x1="29.21" y1="69.215" x2="31.115" y2="71.12" width="0.4064" layer="1" curve="-90"/>
 <wire x1="46.99" y1="66.04" x2="46.99" y2="64.77" width="0.4064" layer="1"/>
 <wire x1="46.99" y1="64.77" x2="47.345" y2="64.77" width="0" layer="19" extent="1-16"/>
@@
 <wire x1="32.385" y1="73.025" x2="31.75" y2="72.39" width="0.6096" layer="1"/>
 <wire x1="31.75" y1="72.39" x2="30.48" y2="72.39" width="0.6096" layer="1"/>
-<wire x1="28.575" y1="70.485" x2="30.48" y2="72.39" width="0.4064" layer="1"/>
+<wire x1="28.575" y1="70.485" x2="30.48" y2="72.39" width="0.4064" layer="1" curve="-90"/>
 <wire x1="47.625" y1="67.945" x2="47.625" y2="67.31" width="0.4064" layer="1"/>
 <wire x1="47.625" y1="67.31" x2="47.845" y2="67.31" width="0" layer="19" extent="1-16"/>
@@
 <wire x1="10.795" y1="43.18" x2="8.89" y2="43.18" width="0.6096" layer="1"/>
 </signal>
+<signal name="N$32">
+<wire x1="79.375" y1="29.21" x2="79.375" y2="24.765" width="0.4064" layer="16"/>
+<wire x1="79.375" y1="24.765" x2="83.82" y2="24.765" width="0.4064" layer="16" curve="180"/>
+<wire x1="83.82" y1="24.765" x2="80.645" y2="26.035" width="0.4064" layer="16" curve="136.397181"/>
+</signal>
+<signal name="N$33">
+<wire x1="78.74" y1="30.48" x2="78.74" y2="24.765" width="0.4064" layer="16"/>
+<wire x1="78.74" y1="24.765" x2="84.455" y2="24.765" width="0.4064" layer="16" curve="180"/>
+<wire x1="84.455" y1="24.765" x2="81.28" y2="27.305" width="0.4064" layer="16" curve="102.680383"/>
+</signal>
+<signal name="N$34">
+<wire x1="78.105" y1="31.75" x2="78.105" y2="24.765" width="0.4064" layer="16"/>
+<wire x1="78.105" y1="24.765" x2="85.09" y2="24.765" width="0.4064" layer="16" curve="180"/>
+<wire x1="85.09" y1="24.765" x2="83.185" y2="27.94" width="0.4064" layer="16" curve="61.927498"/>
+</signal>
+<signal name="N$35">
+<wire x1="80.01" y1="15.875" x2="87.63" y2="15.875" width="0.4064" layer="16"/>
+<wire x1="87.63" y1="15.875" x2="87.63" y2="17.78" width="0.4064" layer="16" curve="180"/>
+<wire x1="87.63" y1="17.78" x2="86.995" y2="16.51" width="0.4064" layer="16" curve="126.869898"/>
+</signal>
+<signal name="N$38">
+<wire x1="81.915" y1="15.24" x2="87.63" y2="15.24" width="0.4064" layer="16"/>
+<wire x1="87.63" y1="15.24" x2="87.63" y2="18.415" width="0.4064" layer="16" curve="180"/>
+<wire x1="87.63" y1="18.415" x2="86.36" y2="16.51" width="0.4064" layer="16" curve="112.619825"/>
+</signal>
+<signal name="N$40">
+<wire x1="77.47" y1="14.605" x2="87.63" y2="14.605" width="0.4064" layer="16"/>
+<wire x1="87.63" y1="14.605" x2="87.63" y2="19.05" width="0.4064" layer="16" curve="180"/>
+<wire x1="87.63" y1="19.05" x2="85.725" y2="16.51" width="0.4064" layer="16" curve="106.260205"/>
+</signal>
+<signal name="N$41">
+<wire x1="80.01" y1="13.97" x2="87.63" y2="13.97" width="0.4064" layer="16"/>
+<wire x1="87.63" y1="13.97" x2="87.63" y2="19.685" width="0.4064" layer="16" curve="180"/>
+<wire x1="87.63" y1="19.685" x2="85.09" y2="16.51" width="0.4064" layer="16" curve="102.680383"/>
+</signal>
+<signal name="N$42">
+<wire x1="75.565" y1="13.335" x2="87.63" y2="13.335" width="0.4064" layer="16"/>
+<wire x1="87.63" y1="13.335" x2="87.63" y2="20.32" width="0.4064" layer="16" curve="180"/>
+<wire x1="87.63" y1="20.32" x2="84.455" y2="16.51" width="0.4064" layer="16" curve="100.388876"/>
+</signal>
+<signal name="N$43">
+<wire x1="81.28" y1="4.445" x2="86.36" y2="4.445" width="0.8128" layer="16"/>
+<wire x1="86.36" y1="4.445" x2="86.36" y2="5.715" width="0.8128" layer="16" curve="180"/>
+<wire x1="86.36" y1="5.715" x2="85.725" y2="5.08" width="0.8128" layer="16" curve="90" cap="flat"/>
+</signal>
+<signal name="N$44">
+<wire x1="79.375" y1="3.175" x2="86.36" y2="3.175" width="0.8128" layer="16"/>
+<wire x1="86.36" y1="3.175" x2="86.36" y2="6.985" width="0.8128" layer="16" curve="180"/>
+<wire x1="86.36" y1="6.985" x2="84.455" y2="5.08" width="0.8128" layer="16" curve="90" cap="flat"/>
+</signal>
+<signal name="N$45">
+<wire x1="78.105" y1="1.905" x2="86.36" y2="1.905" width="0.8128" layer="16"/>
+<wire x1="86.36" y1="1.905" x2="86.36" y2="8.255" width="0.8128" layer="16" curve="180"/>
+<wire x1="86.36" y1="8.255" x2="83.185" y2="5.08" width="0.8128" layer="16" curve="90" cap="flat"/>
+</signal>
+<signal name="N$46">
+<wire x1="86.995" y1="34.29" x2="92.71" y2="34.29" width="0.4064" layer="16"/>
+<wire x1="92.71" y1="34.29" x2="92.71" y2="36.195" width="0.4064" layer="16" curve="180"/>
+<wire x1="92.71" y1="36.195" x2="92.075" y2="34.925" width="0.4064" layer="16" curve="126.869898"/>
+</signal>
+<signal name="N$47">
+<wire x1="85.09" y1="33.655" x2="92.71" y2="33.655" width="0.4064" layer="16"/>
+<wire x1="92.71" y1="33.655" x2="92.71" y2="36.83" width="0.4064" layer="16" curve="180"/>
+<wire x1="92.71" y1="36.83" x2="91.44" y2="36.195" width="0.4064" layer="16" curve="53.130102"/>
+</signal>
+<signal name="N$48">
+<wire x1="83.82" y1="33.02" x2="92.71" y2="33.02" width="0.4064" layer="16"/>
+<wire x1="92.71" y1="33.02" x2="92.71" y2="37.465" width="0.4064" layer="16" curve="180"/>
+<wire x1="92.71" y1="37.465" x2="92.075" y2="37.465" width="0.4064" layer="16"/>
+</signal>
+<signal name="N$49">
+<polygon width="0.4064" layer="1" spacing="0.4064">
+<vertex x="3.81" y="1.905"/>
+<vertex x="63.5" y="1.905"/>
+<vertex x="63.5" y="79.375"/>
+<vertex x="3.81" y="79.375"/>
+</polygon>
+</signal>
 </signals>

Commit message: fixed pours both sides; little logo
Routing:
- added copper zone on layer 1, net +5V
- added copper zone on layer 16, net GND
- removed copper zone on layer 1, net N$49
Changed lines of the file:
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@@
 <wire x1="43.815" y1="65.405" x2="29.21" y2="65.405" width="0.6096" layer="16"/>
 <wire x1="29.21" y1="65.405" x2="26.67" y2="62.865" width="0.6096" layer="16"/>
-<wire x1="57.15" y1="52.07" x2="57.15" y2="49.53" width="0" layer="19" extent="1-1"/>
-<wire x1="10.795" y1="35.56" x2="24.13" y2="60.96" width="0" layer="19" extent="1-1"/>
+<polygon width="0.4064" layer="16">
+<vertex x="3.81" y="78.74"/>
+<vertex x="64.135" y="78.74"/>
+<vertex x="64.135" y="1.27"/>
+<vertex x="3.81" y="1.27"/>
+</polygon>
 </signal>
 <signal name="+5V">
@@
 <wire x1="21.59" y1="28.575" x2="40.005" y2="46.99" width="1.016" layer="16"/>
 <wire x1="40.005" y1="46.99" x2="57.15" y2="46.99" width="1.016" layer="16"/>
-<wire x1="50.8" y1="66.455" x2="50.445" y2="64.77" width="0" layer="19" extent="1-1"/>
-<wire x1="50.445" y1="46.99" x2="50.8" y2="46.99" width="0" layer="19" extent="1-1"/>
-<wire x1="50.445" y1="25.4" x2="50.8" y2="25.4" width="0" layer="19" extent="1-1"/>
-<wire x1="50.445" y1="62.23" x2="50.445" y2="64.77" width="0" layer="19" extent="1-1"/>
-<wire x1="50.445" y1="44.45" x2="50.445" y2="46.99" width="0" layer="19" extent="1-1"/>
-<wire x1="50.8" y1="27.94" x2="50.8" y2="25.4" width="0" layer="19" extent="1-1"/>
-<wire x1="49.945" y1="30.48" x2="50.165" y2="27.94" width="0" layer="19" extent="1-1"/>
-<wire x1="49.945" y1="49.53" x2="50.445" y2="46.99" width="0" layer="19" extent="1-1"/>
-<wire x1="49.945" y1="58.42" x2="50.445" y2="62.23" width="0" layer="19" extent="1-1"/>
-<wire x1="50.445" y1="55.88" x2="49.945" y2="58.42" width="0" layer="19" extent="1-1"/>
-<wire x1="50.445" y1="53.34" x2="50.445" y2="55.88" width="0" layer="19" extent="1-1"/>
-<wire x1="49.945" y1="40.64" x2="50.445" y2="44.45" width="0" layer="19" extent="1-1"/>
-<wire x1="50.445" y1="38.1" x2="49.945" y2="40.64" width="0" layer="19" extent="1-1"/>
-<wire x1="50.445" y1="35.56" x2="50.445" y2="38.1" width="0" layer="19" extent="1-1"/>
 <wire x1="40.005" y1="46.99" x2="40.005" y2="52.07" width="1.016" layer="16"/>
 <wire x1="40.005" y1="52.07" x2="37.465" y2="54.61" width="1.016" layer="16"/>
+<polygon width="0.4064" layer="1" spacing="0.4064">
+<vertex x="3.81" y="1.905"/>
+<vertex x="63.5" y="1.905"/>
+<vertex x="63.5" y="79.375"/>
+<vertex x="3.81" y="79.375"/>
+</polygon>
 </signal>
 <signal name="N$2">
@@
 <wire x1="36.195" y1="58.42" x2="36.195" y2="52.705" width="0.6096" layer="1"/>
 <wire x1="36.195" y1="52.705" x2="37.465" y2="51.435" width="0.6096" layer="1"/>
-<wire x1="37.465" y1="51.435" x2="37.465" y2="50.895" width="0" layer="19" extent="1-16"/>
+<wire x1="37.465" y1="51.435" x2="37.465" y2="50.895" width="0" layer="19" extent="1-1"/>
 </signal>
 <signal name="N$1">
@@
 <wire x1="22.86" y1="34.29" x2="22.86" y2="32.385" width="0.6096" layer="1"/>
 <wire x1="22.86" y1="32.385" x2="23.495" y2="31.75" width="0.6096" layer="1"/>
-<wire x1="23.495" y1="31.75" x2="24.13" y2="31.75" width="0" layer="19" extent="1-16"/>
+<wire x1="23.495" y1="31.75" x2="24.13" y2="31.75" width="0" layer="19" extent="1-1"/>
 </signal>
 <signal name="N$6">
@@
 <wire x1="32.385" y1="48.26" x2="33.655" y2="49.53" width="0.4064" layer="1"/>
 <contactref element="RED4" pad="C"/>
-<wire x1="34.29" y1="49.53" x2="33.655" y2="49.53" width="0" layer="19" extent="1-1"/>
-<wire x1="46.575" y1="41.91" x2="34.29" y2="41.91" width="0" layer="19" extent="1-16"/>
 <wire x1="47.845" y1="40.64" x2="45.085" y2="40.64" width="0.6096" layer="1"/>
 <wire x1="45.085" y1="40.64" x2="43.815" y2="41.91" width="0.6096" layer="1"/>
 <wire x1="43.815" y1="41.91" x2="34.29" y2="41.91" width="0.6096" layer="1"/>
-<wire x1="34.29" y1="41.91" x2="46.575" y2="41.91" width="0" layer="19" extent="1-16"/>
+<wire x1="33.655" y1="49.53" x2="34.29" y2="49.53" width="0" layer="19" extent="1-1"/>
 </signal>
 <signal name="N$21">
@@
 <contactref element="U$2" pad="18"/>
 <contactref element="RED5" pad="C"/>
-<wire x1="33.655" y1="53.34" x2="34.29" y2="53.34" width="0" layer="19" extent="1-1"/>
 <wire x1="34.29" y1="38.1" x2="37.465" y2="38.1" width="0.6096" layer="1"/>
 <wire x1="37.465" y1="38.1" x2="45.085" y2="30.48" width="0.6096" layer="1"/>
 <wire x1="45.085" y1="30.48" x2="47.625" y2="30.48" width="0.6096" layer="1"/>
-<wire x1="47.625" y1="30.48" x2="47.845" y2="30.48" width="0" layer="19" extent="1-16"/>
+<wire x1="33.655" y1="53.34" x2="34.29" y2="53.34" width="0" layer="19" extent="1-1"/>
+<wire x1="47.845" y1="30.48" x2="47.625" y2="30.48" width="0" layer="19" extent="1-1"/>
 </signal>
 <signal name="N$24">
@@
 <contactref element="U$2" pad="19"/>
 <contactref element="GREEN5" pad="C"/>
-<wire x1="33.655" y1="54.61" x2="34.29" y2="54.61" width="0" layer="19" extent="1-1"/>
 <wire x1="34.29" y1="36.83" x2="36.195" y2="36.83" width="0.6096" layer="1"/>
 <wire x1="36.195" y1="36.83" x2="45.085" y2="27.94" width="0.6096" layer="1"/>
 <wire x1="45.085" y1="27.94" x2="47.345" y2="27.94" width="0.6096" layer="1"/>
+<wire x1="33.655" y1="54.61" x2="34.29" y2="54.61" width="0" layer="19" extent="1-1"/>
 </signal>
 <signal name="N$26">
@@
 <wire x1="31.115" y1="57.15" x2="31.115" y2="65.405" width="0.4064" layer="1"/>
 <wire x1="31.115" y1="65.405" x2="33.02" y2="67.31" width="0.4064" layer="1" curve="-90"/>
-<wire x1="33.02" y1="67.31" x2="33.655" y2="67.945" width="0" layer="19" extent="1-16"/>
 <wire x1="47.345" y1="55.88" x2="45.085" y2="55.88" width="0.6096" layer="1"/>
 <wire x1="45.085" y1="55.88" x2="43.18" y2="57.785" width="0.6096" layer="1"/>
@@
 <wire x1="30.48" y1="57.785" x2="30.48" y2="66.675" width="0.4064" layer="1"/>
 <wire x1="30.48" y1="66.675" x2="32.385" y2="68.58" width="0.4064" layer="1" curve="-90"/>
-<wire x1="32.385" y1="68.58" x2="33.655" y2="69.85" width="0" layer="19" extent="1-16"/>
 <wire x1="47.845" y1="58.42" x2="45.085" y2="58.42" width="0.6096" layer="1"/>
 <wire x1="45.085" y1="58.42" x2="44.45" y2="59.055" width="0.6096" layer="1"/>
@@
 <wire x1="24.765" y1="53.34" x2="29.845" y2="58.42" width="0.4064" layer="1"/>
 <wire x1="29.845" y1="58.42" x2="29.845" y2="67.945" width="0.4064" layer="1"/>
-<wire x1="34.29" y1="69.85" x2="47.345" y2="62.23" width="0" layer="19" extent="1-16"/>
 <wire x1="47.345" y1="62.23" x2="46.355" y2="62.23" width="0.6096" layer="1"/>
 <wire x1="46.355" y1="62.23" x2="45.72" y2="62.865" width="0.6096" layer="1"/>
@@
 <wire x1="29.21" y1="69.215" x2="31.115" y2="71.12" width="0.4064" layer="1" curve="-90"/>
 <wire x1="46.99" y1="66.04" x2="46.99" y2="64.77" width="0.4064" layer="1"/>
-<wire x1="46.99" y1="64.77" x2="47.345" y2="64.77" width="0" layer="19" extent="1-16"/>
 </signal>
 <signal name="N$16">
@@
 <wire x1="28.575" y1="70.485" x2="30.48" y2="72.39" width="0.4064" layer="1" curve="-90"/>
 <wire x1="47.625" y1="67.945" x2="47.625" y2="67.31" width="0.4064" layer="1"/>
-<wire x1="47.625" y1="67.31" x2="47.845" y2="67.31" width="0" layer="19" extent="1-16"/>
 </signal>
 <signal name="N$39">
@@
 <wire x1="29.21" y1="51.435" x2="33.655" y2="55.88" width="0.4064" layer="1"/>
 <contactref element="BLUE5" pad="C"/>
-<wire x1="33.655" y1="55.88" x2="34.29" y2="55.88" width="0" layer="19" extent="1-1"/>
 <wire x1="47.345" y1="25.4" x2="45.085" y2="25.4" width="0.6096" layer="1"/>
 <wire x1="45.085" y1="25.4" x2="34.925" y2="35.56" width="0.6096" layer="1"/>
 <wire x1="34.925" y1="35.56" x2="34.29" y2="35.56" width="0.6096" layer="1"/>
+<wire x1="33.655" y1="55.88" x2="34.29" y2="55.88" width="0" layer="19" extent="1-1"/>
 </signal>
 <signal name="N$9">
@@
 <wire x1="92.71" y1="37.465" x2="92.075" y2="37.465" width="0.4064" layer="16"/>
 </signal>
-<signal name="N$49">
-<polygon width="0.4064" layer="1" spacing="0.4064">
-<vertex x="3.81" y="1.905"/>
-<vertex x="63.5" y="1.905"/>
-<vertex x="63.5" y="79.375"/>
-<vertex x="3.81" y="79.375"/>
-</polygon>
-</signal>
 </signals>

Commit message: finished Prototype1, created gerber
Parts:
- moved C2 20.1 mm to (31.1, 35.6)
- moved U$3 18.9 mm to (22.9, 19.7)
- moved BLUE2 18.9 mm to (42.5, 35.6)
- moved BLUE3 18.9 mm to (42.5, 26.7)
- moved BLUE4 18.9 mm to (42.5, 17.8)
- moved GREEN2 18.9 mm to (42.5, 38.1)
- moved GREEN3 18.9 mm to (42.5, 29.2)
- moved GREEN4 18.9 mm to (42.5, 20.3)
- moved GREEN5 18.9 mm to (42.5, 10.2)
- moved R2 18.9 mm to (9.53, 12.7)
- moved R3 18.9 mm to (24.1, 45.1)
- moved RED1 18.9 mm to (42.5, 49.5)
- moved RED2 18.9 mm to (42.5, 40.6)
- moved RED3 18.9 mm to (42.5, 31.8)
- moved RED4 18.9 mm to (42.5, 22.9)
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Connections:
- removed net N$1: C1.2, C2.2, U$2.24
- removed net N$6: C3.2, C4.2, U$3.24
- net +5V: now also C1.2, C2.2, C3.2, C4.2, U$2.24, U$3.24; no longer C1.1, C2.1, C3.1, C4.1
- net GND: now also C1.1, C2.1, C3.1, C4.1, U$2.21, U$3.21
Routing:
- net GND: track 85.6 -> 153.4 mm
- net N$45: track 19.1 -> 0.00 mm
- net N$34: track 17.7 -> 0.00 mm
- net N$33: track 15.5 -> 0.00 mm
- net N$48: track 14.0 -> 0.00 mm
- net N$44: track 13.5 -> 0.00 mm
- net N$32: track 12.3 -> 0.00 mm
- net N$47: track 12.2 -> 0.00 mm
- net N$46: track 9.04 -> 0.00 mm
- net +5V: track 112.2 -> 119.6 mm
- net N$43: track 7.25 -> 0.00 mm
- net N$1: track 6.24 -> 0.00 mm
- net N$6: track 3.81 -> 0.00 mm
- net N$4: track 9.94 -> 12.1 mm
- net N$3: track 6.57 -> 4.49 mm
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Other:
- board size 100 x 80 mm -> 53 x 59.7 mm
- board text added: "BOT"
- board text added: "TOP"
