File: hardware/eagle/prototype2/Prototype1.brd (EAGLE design)
At the start: 53 x 59.7 mm, 18 parts, among them U1 ARDUINO_SHIELDLABEL

Commit message: proto2.zip
Routing:
- net N$39: track 55.3 -> 57.8 mm
- net N$31: track 53.3 -> 55.9 mm
- net N$43: track 57.0 -> 59.5 mm
- net N$33: track 52.7 -> 55.3 mm
- net N$32: track 50.6 -> 53.1 mm
- net N$25: track 31.5 -> 34.0 mm
- net N$34: track 57.3 -> 59.8 mm
- net GND: track 176.0 -> 176.6 mm
