File: hardware/eagle/prototype2/Prototype2.sch (EAGLE design)
At the start: 18 parts, among them U1 ARDUINO_SHIELDLABEL

Commit message: prototype2: resistor values, partlist
Parts:
- R1: value (none) -> 5.6k
- R2: value (none) -> 2.2k
- R3: value (none) -> 50k
- R4: value (none) -> 22k
- R5: value (none) -> 10k
- R6: value (none) -> 100k
Changed lines of the file:
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@@
 <setting verticaltext="up"/>
 </settings>
-<grid distance="0.05" unitdist="inch" unit="inch" style="lines" multiple="1" display="no" altdistance="0.01" altunitdist="inch" altunit="inch"/>
+<grid distance="0.1" unitdist="inch" unit="inch" style="lines" multiple="1" display="no" altdistance="0.01" altunitdist="inch" altunit="inch"/>
 <layers>
 <layer number="1" name="Top" color="4" fill="1" visible="no" active="no"/>
@@
 <part name="U$3" library="CAT4016" deviceset="CAT4016" device=""/>
 <part name="P+3" library="supply1" deviceset="+5V" device=""/>
-<part name="R2" library="rcl" deviceset="R-EU_" device="0204/7"/>
-<part name="R5" library="rcl" deviceset="R-TRIMM" device="3165W"/>
+<part name="R2" library="rcl" deviceset="R-EU_" device="0204/7" value="2.2k"/>
+<part name="R5" library="rcl" deviceset="R-TRIMM" device="3165W" value="10k"/>
 <part name="GND3" library="supply1" deviceset="GND" device=""/>
 <part name="GND4" library="supply1" deviceset="GND" device=""/>
@@
 <part name="U$1" library="CAT4016" deviceset="CAT4016" device=""/>
 <part name="P+2" library="supply1" deviceset="+5V" device=""/>
-<part name="R1" library="rcl" deviceset="R-EU_" device="0204/7"/>
-<part name="R3" library="rcl" deviceset="R-TRIMM" device="3165W"/>
+<part name="R1" library="rcl" deviceset="R-EU_" device="0204/7" value="5.6k"/>
+<part name="R3" library="rcl" deviceset="R-TRIMM" device="3165W" value="50k"/>
 <part name="GND2" library="supply1" deviceset="GND" device=""/>
 <part name="GND5" library="supply1" deviceset="GND" device=""/>
 <part name="C2" library="rcl" deviceset="CPOL-EU" device="A/3216-18W"/>
 <part name="U$2" library="CAT4016" deviceset="CAT4016" device=""/>
-<part name="R4" library="rcl" deviceset="R-EU_" device="0204/7"/>
-<part name="R6" library="rcl" deviceset="R-TRIMM" device="3165W"/>
+<part name="R4" library="rcl" deviceset="R-EU_" device="0204/7" value="22k"/>
+<part name="R6" library="rcl" deviceset="R-TRIMM" device="3165W" value="100k"/>
 <part name="GND6" library="supply1" deviceset="GND" device=""/>
 <part name="GND7" library="supply1" deviceset="GND" device=""/>
